File: hardware/SinglePair-Eth-Gateway/SinglePair-Eth-Gateway.kicad_pcb (KiCad board)
At the start: 4 copper layers, 100 x 54 mm, 119 parts, among them IC401 LDL112PV33R, J201 Conn_01x06_Pin, J202 Conn_01x04, J203 USB_B_Micro, J301 09452812800, J302 Screw_Terminal_01x02, J401 Wuerth-694108301002, T301 74930000, U201 WE-TVS-82400102, U301 WE-TVS-82400102, U302 ADIN1110BCPZ, U401 VXO7803-1000, U501 7499010211A, U502 W5500, U601 TXB0108PWR, Y301 830108212509, Y501 830108212509

Commit message: Change position of values on the Fab layer
Parts:
- FB201, FB202, FB401, FB402, FB403, FB501, FB502: value HH-1M1005-221JT -> BLM18KG121TZ1D
